Commit message: Added cad model for the jump and modified urdf file so that it is correcttly referenced

File: ackermann_vehicle_description/urdf/jump22deg.urdf (robot description, URDF)
Before this commit: robot jump22deg, 1 links, 0 joints
Links:
- link jump22deg_link: geometry collision mesh filename=package://ackermann_vehicle_description/urdf/jump22deg.dae scale=0.01 0.01 0.01; visual mesh filename=package://ackermann_vehicle_description/urdf/jump22deg.dae scale=0.01 0.01 0.01
