Commit message: added 30 deg jump, replaced .dae with .stl files

File: ackermann_vehicle_description/urdf/jump30deg.urdf (robot description, URDF)
Before this commit: robot jump22deg, 1 links, 0 joints
Links:
- removed link jump22deg_link
- added link jump30deg_link, mass 1000000000.0; collision mesh filename=package://ackermann_vehicle_description/urdf/jump30deg.stl scale=0.01 0.01 0.01; visual mesh filename=package://ackermann_vehicle_description/urdf/jump30deg.stl scale=0.01 0.01 0.01
