Commit message: made model more like our robot, getting the world together

File: ackermann_vehicle_description/urdf/em_3905.urdf.xacro (robot description, xacro)
@@ -33,20 +33,8 @@
   <!-- chassis_length is measured along the x axis, chassis_width
        along the y axis, and chassis_height along the z axis. -->
-  <xacro:property name="chassis_length" value="0.258"/>
-  <xacro:property name="chassis_width" value="0.168"/>
-  <xacro:property name="chassis_height" value="0.01"/>
-  <xacro:property name="chassis_mass" value="2.788"/>
-  <!-- battery_dist is the distance between the inner edges of the
-       batteries. battery_comp_depth is the battery compartment depth.
-       battery_length is measured along the x axis, battery_width
-       along the y axis, and battery_height along the z axis. -->
-  <xacro:property name="battery_x_offset" value="0.055"/>
-  <xacro:property name="battery_dist" value="0.065"/>
-  <xacro:property name="battery_comp_depth" value="0.02"/>
-  <xacro:property name="battery_comp_angle" value="0.34906585"/>
-  <xacro:property name="battery_length" value="0.16"/>
-  <xacro:property name="battery_width" value="0.047"/>
-  <xacro:property name="battery_height" value="0.024"/>
-  <xacro:property name="battery_mass" value="0.5025"/>
+  <xacro:property name="chassis_length" value="0.90"/>
+  <xacro:property name="chassis_width" value="0.20"/>
+  <xacro:property name="chassis_height" value="0.25"/>
+  <xacro:property name="chassis_mass" value="19.555"/>
   <!-- hub_dia and tire_dia are the diameters of the hub and tire,
        respectively. hex_hub_depth is the distance that the hex hub is
@@ -54,23 +42,29 @@
        is a "zero offset" wheel. hex_hub_depth = tire_width / 2 -
        axle_length. -->
-  <xacro:property name="hub_dia" value="0.09652"/>
-  <xacro:property name="tire_dia" value="0.14605"/>
-  <xacro:property name="tire_width" value="0.0889"/>
-  <xacro:property name="hex_hub_depth" value="0.01445"/>
-  <xacro:property name="wheel_mass" value="0.29"/>
+  <xacro:property name="hub_dia" value="0.024"/>
+  <xacro:property name="tire_dia" value="0.19"/>
+  <xacro:property name="hex_hub_depth" value="0.035"/>
+  <xacro:property name="front_tire_width" value="0.06"/>
+  <xacro:property name="front_wheel_mass" value="0.495"/>
+  <xacro:property name="rear_tire_width" value="0.07"/>
+  <xacro:property name="rear_wheel_mass" value="0.660"/>
   <!-- hex_hub_dist is the distance between left and right hex hubs when
        the shock absorbers are fully extended. axle_length is the distance
        from a U joint to the corresponding hex hub. wheel_travel is the
        vertical wheel travel. -->
-  <xacro:property name="wheelbase" value="0.335"/>
-  <xacro:property name="hex_hub_dist" value="0.365"/>
+  <xacro:property name="wheelbase" value="0.570"/>
+  <xacro:property name="hex_hub_dist" value="0.4"/>
   <xacro:property name="axle_length" value="0.03"/>
-  <xacro:property name="wheel_travel" value="0.084"/>
-  <xacro:property name="shock_z_offset" value="0.0655"/>
+  <xacro:property name="wheel_travel" value="0.1"/>
+  <xacro:property name="shock_z_offset" value="0.11"/>
+  <xacro:property name="front_wheel_travel" value="0.1"/>
+  <xacro:property name="front_shock_z_offset" value="0.1"/>
+  <xacro:property name="rear_wheel_travel" value="0.1"/>
+  <xacro:property name="rear_shock_z_offset" value="0.12"/>
   <!-- shock_eff_limit is 2 * ((shock_stroke / 2) * shock_spring_constant) N.
        shock_stroke is 0.028575 meters. shock_spring_constant, an approximation
        of a Traxxas Ultra Shock shock absorber spring's constant, is
        437.817 N/m. -->
-  <xacro:property name="shock_eff_limit" value="12.5106"/>
+  <xacro:property name="shock_eff_limit" value="157.6141515"/>
   <xacro:property name="shock_vel_limit" value="1000"/>
   <!-- The specifications for a Titan(R) 550 motor could not be found, so the
@@ -85,15 +79,15 @@
        max_speed = 40 mph (30+ mph) = 17.8816 m/s
        axle_vel_limit = (2 * pi) * (max_speed / (pi * tire_dia)) =
-         244.8696 rad/s -->
-  <xacro:property name="axle_eff_limit" value="5.12766"/>
-  <xacro:property name="axle_vel_limit" value="244.8696"/>
+         244.8696 rad/s
+       60mph = 26.82 m/s
+       2*26.82/0.19 = 282.315789474
+          -->
+  <xacro:property name="axle_eff_limit" value="5"/>
+  <xacro:property name="axle_vel_limit" value="282.315789474"/>
   <!-- These constants are used to simulate a Traxxas 2056 servo operated at
        6 V. servo_stall_torque is measured in N m. servo_no_load_speed is
        measured in rad/s. -->
-  <xacro:property name="servo_stall_torque" value="0.5649"/>
-  <xacro:property name="servo_no_load_speed" value="4.553"/>
-  <material name="battery_mat">
-    <color rgba="0 0 1 1"/>
-  </material>
+  <xacro:property name="servo_stall_torque" value="3.432620346181713"/>
+  <xacro:property name="servo_no_load_speed" value="6.553"/>
   <material name="chassis_mat">
     <color rgba="0.5 0.5 0.5 1"/>
@@ -110,18 +104,4 @@
     </inertial>
   </xacro:macro>
-  <!-- Inertia of a solid cuboid. Width is measured along the x axis, depth
-       along the y axis, and height along the z axis. -->
-  <xacro:macro name="solid_cuboid_inertial"
-               params="width depth height mass *origin">
-    <inertial>
-      <xacro:insert_block name="origin"/>
-      <mass value="${mass}"/>
-      <inertia ixx="${mass * (depth * depth + height * height) / 12}"
-               ixy="0" ixz="0"
-               iyy="${mass * (width * width + height * height) / 12}"
-               iyz="0"
-               izz="${mass * (width * width + depth * depth) / 12}"/>
-    </inertial>
-  </xacro:macro>
   <!-- Inertia of a thick-walled cylindrical tube with open ends. Height is
        measured along the z axis, which is the tube's axis. inner_rad and
@@ -134,52 +114,9 @@
                     outer_rad * outer_rad) + height * height)}"
                ixy="0" ixz="0"
-               iyy="${(1 / 12) * mass * (3 * (inner_rad * inner_rad +
-                    outer_rad * outer_rad) + height * height)}"
+               iyy="0.0095910648"
                iyz="0"
                izz="${mass * (inner_rad * inner_rad +
                     outer_rad * outer_rad) / 2}"/>
     </inertial>
-  </xacro:macro>
-  <!-- Battery -->
-  <xacro:macro name="battery" params="prefix reflect">
-    <joint name="chassis_to_${prefix}_battery" type="fixed">
-      <parent link="chassis"/>
-      <child link="${prefix}_battery_offset"/>
-      <origin xyz="${battery_x_offset - battery_length / 2}
-                   ${reflect * battery_dist / 2}
-                   0"
-              rpy="${reflect * battery_comp_angle} 0 0"/>
-    </joint>
-    <link name="${prefix}_battery_offset">
-      <xacro:null_inertial/>
-    </link>
-    <joint name="offset_to_${prefix}_battery" type="fixed">
-      <parent link="${prefix}_battery_offset"/>
-      <child link="${prefix}_battery"/>
-      <origin xyz="0
-                   ${reflect * battery_width / 2}
-                   ${(battery_height / 2) - battery_comp_depth}"/>
-    </joint>
-    <link name="${prefix}_battery">
-      <visual>
-        <geometry>
-          <box size="${battery_length} ${battery_width} ${battery_height}"/>
-        </geometry>
-        <material name="battery_mat"/>
-      </visual>
-      <collision>
-        <geometry>
-          <box size="${battery_length} ${battery_width} ${battery_height}"/>
-        </geometry>
-      </collision>
-      <xacro:solid_cuboid_inertial
-         width="${battery_length}" depth="${battery_width}"
-         height="${battery_height}" mass="${battery_mass}">
-        <origin/>
-      </xacro:solid_cuboid_inertial>
-    </link>
-    <gazebo reference="${prefix}_battery">
-      <material>Gazebo/Blue</material>
-    </gazebo>
   </xacro:macro>
   <!-- Shock absorber -->
@@ -191,5 +128,5 @@
       <origin xyz="${fr_reflect * wheelbase / 2}
                    ${lr_reflect * ((hex_hub_dist / 2) - axle_length)}
-                   ${(wheel_travel / 2) - shock_z_offset}"/>
+                   ${-chassis_height/2 + (wheel_travel / 2) - shock_z_offset}"/>
       <axis xyz="0 0 -1"/>
       <limit lower="${-wheel_travel / 2}" upper="${wheel_travel / 2}"
@@ -210,5 +147,5 @@
   </xacro:macro>
   <!-- The "wheel" macro defines an axle carrier, axle, and wheel. -->
-  <xacro:macro name="wheel" params="lr_prefix fr_prefix lr_reflect">
+  <xacro:macro name="wheel" params="lr_prefix fr_prefix lr_reflect tire_width wheel_mass">
     <link name="${lr_prefix}_${fr_prefix}_axle_carrier">
       <xacro:null_inertial/>
@@ -238,7 +175,7 @@
       <visual>
         <origin xyz="0
-                     ${lr_reflect * (axle_length - (tire_width /
-                     2 - hex_hub_depth))}
-                     0"/>
+                     0
+                     0
+                     "/>
         <geometry>
           <cylinder radius="${tire_dia / 2}" length="${tire_width}"/>
@@ -248,10 +185,20 @@
       <collision>
         <origin xyz="0
-                     ${lr_reflect * (axle_length - (tire_width /
-                     2 - hex_hub_depth))}
-                     0"/>
+                     0
+                     0
+                     "/>
         <geometry>
           <cylinder radius="${tire_dia / 2}" length="${tire_width}"/>
         </geometry>
+        <surface>
+          <friction>
+            <ode>
+              <mu>0.0</mu>
+              <mu2>0.0</mu2>
+              <slip1>0.0</slip1>
+              <slip2>0.0</slip2>
+            </ode>
+          </friction>
+        </surface>
       </collision>
       <xacro:thick_walled_tube_inertial
@@ -265,5 +212,5 @@
   <!-- Front wheel -->
   <xacro:macro name="front_wheel"
-               params="lr_prefix fr_prefix lr_reflect fr_reflect">
+               params="lr_prefix fr_prefix lr_reflect fr_reflect tire_width wheel_mass">
     <xacro:shock lr_prefix="${lr_prefix}" fr_prefix="${fr_prefix}"
                  lr_reflect="${lr_reflect}" fr_reflect="${fr_reflect}"
@@ -292,14 +239,16 @@
     </transmission>
     <xacro:wheel lr_prefix="${lr_prefix}" fr_prefix="${fr_prefix}"
-                 lr_reflect="${lr_reflect}"/>
+                 lr_reflect="${lr_reflect}" tire_width="${tire_width}"
+                 wheel_mass="${wheel_mass}"/>
   </xacro:macro>
   <!-- Rear wheel -->
   <xacro:macro name="rear_wheel"
-               params="lr_prefix fr_prefix lr_reflect fr_reflect">
+               params="lr_prefix fr_prefix lr_reflect fr_reflect tire_width wheel_mass">
     <xacro:shock lr_prefix="${lr_prefix}" fr_prefix="${fr_prefix}"
                  lr_reflect="${lr_reflect}" fr_reflect="${fr_reflect}"
                  child="${lr_prefix}_${fr_prefix}_axle_carrier"/>
     <xacro:wheel lr_prefix="${lr_prefix}" fr_prefix="${fr_prefix}"
-                 lr_reflect="${lr_reflect}"/>
+                 lr_reflect="${lr_reflect}" tire_width="${tire_width}"
+                 wheel_mass="${wheel_mass}"/>
   </xacro:macro>
   <!-- base_link must have geometry so that its axes can be displayed in
@@ -331,9 +280,12 @@
       </geometry>
     </collision>
-    <xacro:solid_cuboid_inertial
-        width="${chassis_length}" depth="${chassis_width}"
-        height="${chassis_height}" mass="${chassis_mass}">
-      <origin xyz="0 0 ${-chassis_height / 2}"/>
-    </xacro:solid_cuboid_inertial>
+    <inertial>
+      <mass value="${chassis_mass}"/>
+      <inertia ixx="0.3881755275"
+               ixy="0" ixz="0"
+               iyy="1.1310597718"
+               iyz="0"
+               izz="1.1243832479"/>
+    </inertial>
   </link>
   <gazebo reference="chassis">
@@ -344,16 +296,21 @@
     <child link="chassis"/>
   </joint>
-  <!-- Batteries -->
-  <xacro:battery prefix="left" reflect="1"/>
-  <xacro:battery prefix="right" reflect="-1"/>
   <!-- Wheels -->
   <xacro:front_wheel lr_prefix="left" fr_prefix="front"
-                     lr_reflect="1" fr_reflect="1"/>
+                     lr_reflect="1" fr_reflect="1"
+                     tire_width="${front_tire_width}"
+                     wheel_mass="${front_wheel_mass}"/>
   <xacro:front_wheel lr_prefix="right" fr_prefix="front"
-                     lr_reflect="-1" fr_reflect="1"/>
+                     lr_reflect="-1" fr_reflect="1"
+                     tire_width="${front_tire_width}"
+                     wheel_mass="${front_wheel_mass}"/>
   <xacro:rear_wheel lr_prefix="left" fr_prefix="rear"
-                    lr_reflect="1" fr_reflect="-1"/>
+                    lr_reflect="1" fr_reflect="-1"
+                    tire_width="${rear_tire_width}"
+                    wheel_mass="${rear_wheel_mass}"/>
   <xacro:rear_wheel lr_prefix="right" fr_prefix="rear"
-                    lr_reflect="-1" fr_reflect="-1"/>
+                    lr_reflect="-1" fr_reflect="-1"
+                    tire_width="${rear_tire_width}"
+                    wheel_mass="${rear_wheel_mass}"/>
   <gazebo>
     <plugin name="gazebo_ros_control" filename="libgazebo_ros_control.so"/>

Commit message: added 5sc chassis model and updated some values

File: ackermann_vehicle_description/urdf/em_3905.urdf.xacro (robot description, xacro)
@@ -27,5 +27,5 @@
 limitations under the License.
 -->
-<robot name="em_3905" xmlns:xacro="http://www.ros.org/wiki/xacro">
+<robot name="hpi_baja" xmlns:xacro="http://www.ros.org/wiki/xacro">
   <!-- Degree-to-radian conversions -->
   <xacro:property name="degrees_45" value="0.785398163"/>
@@ -174,38 +174,25 @@
     <link name="${lr_prefix}_${fr_prefix}_wheel">
       <visual>
-        <origin xyz="0
-                     0
-                     0
-                     "/>
+        <origin xyz="0 0 0"/>
         <geometry>
-          <cylinder radius="${tire_dia / 2}" length="${tire_width}"/>
+          <cylinder radius="${tire_dia / 2.0}" length="${tire_width}"/>
         </geometry>
         <material name="tire_mat"/>
       </visual>
-      <collision>
-        <origin xyz="0
-                     0
-                     0
-                     "/>
+      <collision name="collision">
+        <origin xyz="0 0 0"/>
         <geometry>
-          <cylinder radius="${tire_dia / 2}" length="${tire_width}"/>
+          <cylinder radius="${tire_dia / 2.0}" length="${tire_width}"/>
         </geometry>
-        <surface>
-          <friction>
-            <ode>
-              <mu>0.0</mu>
-              <mu2>0.0</mu2>
-              <slip1>0.0</slip1>
-              <slip2>0.0</slip2>
-            </ode>
-          </friction>
-        </surface>
       </collision>
       <xacro:thick_walled_tube_inertial
-          inner_rad="${hub_dia / 2}" outer_rad="${tire_dia / 2}"
+          inner_rad="${hub_dia / 2.0}" outer_rad="${tire_dia / 2.0}"
           height="${tire_width}" mass="${wheel_mass}"/>
     </link>
     <gazebo reference="${lr_prefix}_${fr_prefix}_wheel">
       <material>Gazebo/Black</material>
+      <mu1>0.4</mu1>
+      <mu2>0.6</mu2>
+<!--      <fdir1>1.0 0.0 0.0</fdir1> -->
     </gazebo>
   </xacro:macro>
@@ -268,7 +255,8 @@
   <link name="chassis">
     <visual>
-      <origin xyz="0 0 ${-chassis_height / 2}"/>
+      <origin xyz="${-chassis_length/2 + 0.1} 0 ${-chassis_height}"/>
       <geometry>
-        <box size="${chassis_length} ${chassis_width} ${chassis_height}"/>
+        <mesh filename="package://ackermann_vehicle_description/urdf/5scChassis.stl" scale="0.01 0.01 0.01" />
+        <!-- <box size="${chassis_length} ${chassis_width} ${chassis_height}"/> -->
       </geometry>
       <material name="chassis_mat"/>
@@ -282,9 +270,9 @@
     <inertial>
       <mass value="${chassis_mass}"/>
-      <inertia ixx="0.3881755275"
+      <inertia ixx="0.00003881755275"
                ixy="0" ixz="0"
-               iyy="1.1310597718"
+               iyy="0.00011310597718"
                iyz="0"
-               izz="1.1243832479"/>
+               izz="0.0001243832479"/>
     </inertial>
   </link>

Commit message: improved chassis model, updated vehicle params to be more realistic, added node to control vehicle with joystick

File: ackermann_vehicle_description/urdf/em_3905.urdf.xacro (robot description, xacro)
@@ -30,9 +30,10 @@
   <!-- Degree-to-radian conversions -->
   <xacro:property name="degrees_45" value="0.785398163"/>
+  <xacro:property name="degrees_25" value="0.436332313"/>
   <xacro:property name="degrees_90" value="1.57079633"/>
   <!-- chassis_length is measured along the x axis, chassis_width
        along the y axis, and chassis_height along the z axis. -->
   <xacro:property name="chassis_length" value="0.90"/>
-  <xacro:property name="chassis_width" value="0.20"/>
+  <xacro:property name="chassis_width" value="0.25"/>
   <xacro:property name="chassis_height" value="0.25"/>
   <xacro:property name="chassis_mass" value="19.555"/>
@@ -58,6 +59,6 @@
   <xacro:property name="wheel_travel" value="0.1"/>
   <xacro:property name="shock_z_offset" value="0.11"/>
-  <xacro:property name="front_wheel_travel" value="0.1"/>
-  <xacro:property name="front_shock_z_offset" value="0.1"/>
+  <xacro:property name="front_wheel_travel" value="0.12"/>
+  <xacro:property name="front_shock_z_offset" value="0.09"/>
   <xacro:property name="rear_wheel_travel" value="0.1"/>
   <xacro:property name="rear_shock_z_offset" value="0.12"/>
@@ -83,5 +84,5 @@
        2*26.82/0.19 = 282.315789474
           -->
-  <xacro:property name="axle_eff_limit" value="5"/>
+  <xacro:property name="axle_eff_limit" value="7"/>
   <xacro:property name="axle_vel_limit" value="282.315789474"/>
   <!-- These constants are used to simulate a Traxxas 2056 servo operated at
@@ -89,5 +90,5 @@
        measured in rad/s. -->
   <xacro:property name="servo_stall_torque" value="3.432620346181713"/>
-  <xacro:property name="servo_no_load_speed" value="6.553"/>
+  <xacro:property name="servo_no_load_speed" value="6.98131700798"/>
   <material name="chassis_mat">
     <color rgba="0.5 0.5 0.5 1"/>
@@ -127,9 +128,10 @@
       <child link="${child}"/>
       <origin xyz="${fr_reflect * wheelbase / 2}
-                   ${lr_reflect * ((hex_hub_dist / 2) - axle_length)}
+                   ${lr_reflect * ((hex_hub_dist / 2))}
                    ${-chassis_height/2 + (wheel_travel / 2) - shock_z_offset}"/>
       <axis xyz="0 0 -1"/>
       <limit lower="${-wheel_travel / 2}" upper="${wheel_travel / 2}"
              effort="${shock_eff_limit}" velocity="${shock_vel_limit}"/>
+      <dynamics damping="0.1" friction="0.0"/>
     </joint>
     <transmission name="${lr_prefix}_${fr_prefix}_shock_trans">
@@ -192,6 +194,6 @@
     <gazebo reference="${lr_prefix}_${fr_prefix}_wheel">
       <material>Gazebo/Black</material>
-      <mu1>0.4</mu1>
-      <mu2>0.6</mu2>
+      <mu1>0.45</mu1>
+      <mu2>0.5</mu2>
 <!--      <fdir1>1.0 0.0 0.0</fdir1> -->
     </gazebo>
@@ -210,5 +212,5 @@
       <child link="${lr_prefix}_${fr_prefix}_axle_carrier"/>
       <axis xyz="0 0 1"/>
-      <limit lower="${-degrees_45}" upper="${degrees_45}"
+      <limit lower="${-degrees_25}" upper="${degrees_25}"
              effort="${servo_stall_torque}" velocity="${servo_no_load_speed}"/>
     </joint>
@@ -255,5 +257,5 @@
   <link name="chassis">
     <visual>
-      <origin xyz="${-chassis_length/2 + 0.1} 0 ${-chassis_height}"/>
+      <origin xyz="${-chassis_length/2 + 0.08} 0 ${-chassis_height}"/>
       <geometry>
         <mesh filename="package://ackermann_vehicle_description/urdf/5scChassis.stl" scale="0.01 0.01 0.01" />
@@ -263,16 +265,17 @@
     </visual>
     <collision>
-      <origin xyz="0 0 ${-chassis_height / 2}"/>
+      <origin xyz="${-chassis_length/2 + 0.08} 0 ${-chassis_height}"/>
       <geometry>
-        <box size="${chassis_length} ${chassis_width} ${chassis_height}"/>
+        <mesh filename="package://ackermann_vehicle_description/urdf/5scChassis.stl" scale="0.01 0.01 0.01" />
+        <!-- <box size="${chassis_length} ${chassis_width} ${chassis_height}"/> -->
       </geometry>
     </collision>
     <inertial>
       <mass value="${chassis_mass}"/>
-      <inertia ixx="0.00003881755275"
+      <inertia ixx="0.003881755275"
                ixy="0" ixz="0"
-               iyy="0.00011310597718"
+               iyy="0.011310597718"
                iyz="0"
-               izz="0.0001243832479"/>
+               izz="0.01243832479"/>
     </inertial>
   </link>

Commit message: added dmaping properly to the shocks, removed uit from the d term in the shock position controller, jittering has stopped

File: ackermann_vehicle_description/urdf/em_3905.urdf.xacro (robot description, xacro)
@@ -133,5 +133,5 @@
       <limit lower="${-wheel_travel / 2}" upper="${wheel_travel / 2}"
              effort="${shock_eff_limit}" velocity="${shock_vel_limit}"/>
-      <dynamics damping="0.1" friction="0.0"/>
+      <dynamics damping="50" friction="0.0"/>
     </joint>
     <transmission name="${lr_prefix}_${fr_prefix}_shock_trans">
@@ -196,4 +196,6 @@
       <mu1>0.4</mu1>
       <mu2>0.5</mu2>
+      <kp  value="10000000.0" />
+      <kd  value="1.0" />
 <!--      <fdir1>1.0 0.0 0.0</fdir1> -->
     </gazebo>
@@ -313,8 +315,10 @@
       <rpyOffset>0 0 0</rpyOffset>
       <xyzOffset>0 0 0</xyzOffset>
-      <accelDrift>0.1 0.1 0.1</accelDrift>
-      <accelGaussianNoise>0.05 0.05 0.03</accelGaussianNoise>
+      <accelDrift>0.001 0.001 0.001</accelDrift>
+      <accelGaussianNoise>0.001 0.001 0.001</accelGaussianNoise>
       <rateDrift>0.01 0.01 0.01</rateDrift>
       <rateGaussianNoise>0.05 0.05 0.015</rateGaussianNoise>
+      <headingDrift>0.001 0.001 0.001</headingDrift>
+      <headingGaussianNoise>0.001 0.001 0.0005</headingGaussianNoise>
     </plugin>
     <plugin name="gps" filename="libhector_gazebo_ros_gps.so">
@@ -324,7 +328,7 @@
       <topicName>fix</topicName>
       <velocityTopicName>fix_velocity</velocityTopicName>
-      <referenceLatitude>49.860246</referenceLatitude>
-      <referenceLongitude>8.687077</referenceLongitude>
-      <drift>5.0 5.0 5.0</drift>
+      <referenceLatitude>33.774497</referenceLatitude>
+      <referenceLongitude>-84.405001</referenceLongitude>
+      <drift>0.3 0.3 0.3</drift>
       <gaussianNoise>0.01 0.01 0.01</gaussianNoise>
       <velocityDrift>0 0 0</velocityDrift>

Commit message: trying to separate jump spawning into world file

File: ackermann_vehicle_description/urdf/em_3905.urdf.xacro (robot description, xacro)
@@ -133,5 +133,5 @@
       <limit lower="${-wheel_travel / 2}" upper="${wheel_travel / 2}"
              effort="${shock_eff_limit}" velocity="${shock_vel_limit}"/>
-      <dynamics damping="50" friction="0.0"/>
+      <dynamics damping="65" friction="0.0"/>
     </joint>
     <transmission name="${lr_prefix}_${fr_prefix}_shock_trans">
