Commit message: Added track boundaries and working to add cameras to model

File: ackermann_vehicle_description/urdf/em_3905.urdf.xacro (robot description, xacro)
@@ -195,5 +195,5 @@
       <material>Gazebo/Black</material>
       <mu1>0.45</mu1>
-      <mu2>0.55</mu2>
+      <mu2>0.5</mu2>
       <kp  value="10000000.0" />
       <kd  value="1.0" />
@@ -284,4 +284,6 @@
   <gazebo reference="chassis">
     <material>Gazebo/Grey</material>
+    <mu1>0.3</mu1>
+    <mu2>0.3</mu2>
   </gazebo>
   <joint name="base_link_to_chasis" type="fixed">
@@ -289,4 +291,89 @@
     <child link="chassis"/>
   </joint>
+  <joint name="camera_joint" type="fixed">
+    <axis xyz="0 0.08 0.05" />
+    <origin xyz="0.2 0 0" rpy="0 0 0"/>
+    <parent link="base_link"/>
+    <child link="camera_link"/>
+  </joint>
+  <!-- Camera -->
+  <link name="camera_link">
+    <collision>
+      <origin xyz="0 0 0" rpy="0 0 0"/>
+      <geometry>
+    <box size="0.05 0.05 0.05"/>
+      </geometry>
+    </collision>
+<!--    <visual>
+      <origin xyz="0 0 0" rpy="0 0 0"/>
+      <geometry>
+    <box size="0.05 0.05 0.05"/>
+      </geometry>
+      <material name="red"/>
+    </visual>
+    <inertial>
+      <mass value="1e-5" />
+      <origin xyz="0 0 0" rpy="0 0 0"/>
+      <inertia ixx="1e-6" ixy="0" ixz="0" iyy="1e-6" iyz="0" izz="1e-6" />
+    </inertial>
+-->
+  </link>
+  <!-- camera -->
+  <gazebo reference="camera_link">
+    <sensor type="multicamera" name="stereo_camera">
+      <update_rate>30.0</update_rate>
+      <camera name="left">
+        <pose>0 0.07 0 0 0 0</pose>
+        <horizontal_fov>1.3962634</horizontal_fov>
+        <image>
+          <width>1280</width>
+          <height>1024</height>
+          <format>R8G8B8</format>
+        </image>
+        <clip>
+          <near>0.02</near>
+          <far>300</far>
+        </clip>
+        <noise>
+          <type>gaussian</type>
+          <mean>0.0</mean>
+          <stddev>0.009</stddev>
+        </noise>
+      </camera>
+      <camera name="right">
+        <pose>0 -0.07 0 0 0 0</pose>
+        <horizontal_fov>2.5</horizontal_fov>
+        <image>
+          <width>1280</width>
+          <height>1024</height>
+          <format>R8G8B8</format>
+        </image>
+        <clip>
+          <near>0.02</near>
+          <far>300</far>
+        </clip>
+        <noise>
+          <type>gaussian</type>
+          <mean>0.0</mean>
+          <stddev>0.009</stddev>
+        </noise>
+      </camera>
+      <plugin name="stereo_camera_controller" filename="libgazebo_ros_multicamera.so">
+        <alwaysOn>true</alwaysOn>
+        <updateRate>60.0</updateRate>
+        <cameraName>camera</cameraName>
+        <imageTopicName>image_raw</imageTopicName>
+        <cameraInfoTopicName>camera_info</cameraInfoTopicName>
+        <frameName>left_camera_optical_frame</frameName>
+        <!--<rightFrameName>right_camera_optical_frame</rightFrameName>-->
+        <hackBaseline>0.14</hackBaseline>
+        <distortionK1>0.0</distortionK1>
+        <distortionK2>0.0</distortionK2>
+        <distortionK3>0.0</distortionK3>
+        <distortionT1>0.0</distortionT1>
+        <distortionT2>0.0</distortionT2>
+      </plugin>
+    </sensor>
+  </gazebo>
   <!-- Wheels -->
   <xacro:front_wheel lr_prefix="left" fr_prefix="front"

Commit message: Updated most camera parameters to match our actual setup, only issue is that  multi-camera setup requires same calibration matrix for each camera even if different FOV (doenst make sense to me). Image Topics are mapped to those published by the actual platform

File: ackermann_vehicle_description/urdf/em_3905.urdf.xacro (robot description, xacro)
@@ -292,6 +292,6 @@
   </joint>
   <joint name="camera_joint" type="fixed">
-    <axis xyz="0 0.08 0.05" />
-    <origin xyz="0.2 0 0" rpy="0 0 0"/>
+    <axis xyz="0 0 0" />
+    <origin xyz="0.12 0 0.05" rpy="0 0 0"/>
     <parent link="base_link"/>
     <child link="camera_link"/>
@@ -302,11 +302,11 @@
       <origin xyz="0 0 0" rpy="0 0 0"/>
       <geometry>
-    <box size="0.05 0.05 0.05"/>
+    <box size="0.02 0.02 0.02"/>
       </geometry>
     </collision>
-<!--    <visual>
+    <visual>
       <origin xyz="0 0 0" rpy="0 0 0"/>
       <geometry>
-    <box size="0.05 0.05 0.05"/>
+    <box size="0.02 0.02 0.02"/>
       </geometry>
       <material name="red"/>
@@ -317,5 +317,4 @@
       <inertia ixx="1e-6" ixy="0" ixz="0" iyy="1e-6" iyz="0" izz="1e-6" />
     </inertial>
--->
   </link>
   <!-- camera -->
@@ -342,6 +341,6 @@
       </camera>
       <camera name="right">
-        <pose>0 -0.07 0 0 0 0</pose>
-        <horizontal_fov>2.5</horizontal_fov>
+        <pose>0.02 -0.07 0 0 0 0</pose>
+        <horizontal_fov>3.0</horizontal_fov>
         <image>
           <width>1280</width>
@@ -368,8 +367,8 @@
         <!--<rightFrameName>right_camera_optical_frame</rightFrameName>-->
         <hackBaseline>0.14</hackBaseline>
-        <distortionK1>0.0</distortionK1>
-        <distortionK2>0.0</distortionK2>
-        <distortionK3>0.0</distortionK3>
-        <distortionT1>0.0</distortionT1>
+        <distortionK1>-0.212652</distortionK1>
+        <distortionK2>0.085434</distortionK2>
+        <distortionK3>-0.000165</distortionK3>
+        <distortionT1>-0.000336</distortionT1>
         <distortionT2>0.0</distortionT2>
       </plugin>

Commit message: Updated friction coefficients for models, making vehicle model more accurate

File: ackermann_vehicle_description/urdf/em_3905.urdf.xacro (robot description, xacro)
@@ -84,5 +84,6 @@
        2*26.82/0.19 = 282.315789474
           -->
-  <xacro:property name="axle_eff_limit" value="7"/>
+  <xacro:property name="front_axle_eff_limit" value="2"/>
+  <xacro:property name="rear_axle_eff_limit" value="7"/>
   <xacro:property name="axle_vel_limit" value="282.315789474"/>
   <!-- These constants are used to simulate a Traxxas 2056 servo operated at
@@ -149,5 +150,5 @@
   </xacro:macro>
   <!-- The "wheel" macro defines an axle carrier, axle, and wheel. -->
-  <xacro:macro name="wheel" params="lr_prefix fr_prefix lr_reflect tire_width wheel_mass">
+  <xacro:macro name="wheel" params="lr_prefix fr_prefix lr_reflect tire_width wheel_mass axle_eff_limit">
     <link name="${lr_prefix}_${fr_prefix}_axle_carrier">
       <xacro:null_inertial/>
@@ -161,5 +162,10 @@
       <axis xyz="0 0 -1"/>
       <limit effort="${axle_eff_limit}" velocity="${axle_vel_limit}"/>
+      <dynamics damping="0.015" friction="0.0"/>
     </joint>
+<!--    <gazebo reference="${lr_prefix}_${fr_prefix}_axle">
+      <dampingFactor>0.8</dampingFactor>
+    </gazebo>
+-->
     <transmission name="${lr_prefix}_${fr_prefix}_axle_trans">
       <type>transmission_interface/SimpleTransmission</type>
@@ -194,14 +200,14 @@
     <gazebo reference="${lr_prefix}_${fr_prefix}_wheel">
       <material>Gazebo/Black</material>
-      <mu1>0.45</mu1>
-      <mu2>0.5</mu2>
+      <mu1>0.5</mu1>
+      <mu2>0.45</mu2>
       <kp  value="10000000.0" />
       <kd  value="1.0" />
-<!--      <fdir1>1.0 0.0 0.0</fdir1> -->
     </gazebo>
   </xacro:macro>
   <!-- Front wheel -->
   <xacro:macro name="front_wheel"
-               params="lr_prefix fr_prefix lr_reflect fr_reflect tire_width wheel_mass">
+               params="lr_prefix fr_prefix lr_reflect fr_reflect tire_width
+                       wheel_mass axle_eff_limit">
     <xacro:shock lr_prefix="${lr_prefix}" fr_prefix="${fr_prefix}"
                  lr_reflect="${lr_reflect}" fr_reflect="${fr_reflect}"
@@ -231,9 +237,11 @@
     <xacro:wheel lr_prefix="${lr_prefix}" fr_prefix="${fr_prefix}"
                  lr_reflect="${lr_reflect}" tire_width="${tire_width}"
-                 wheel_mass="${wheel_mass}"/>
+                 wheel_mass="${wheel_mass}"
+                 axle_eff_limit="${axle_eff_limit}"/>
   </xacro:macro>
   <!-- Rear wheel -->
   <xacro:macro name="rear_wheel"
-               params="lr_prefix fr_prefix lr_reflect fr_reflect tire_width wheel_mass">
+               params="lr_prefix fr_prefix lr_reflect fr_reflect tire_width
+                       wheel_mass axle_eff_limit">
     <xacro:shock lr_prefix="${lr_prefix}" fr_prefix="${fr_prefix}"
                  lr_reflect="${lr_reflect}" fr_reflect="${fr_reflect}"
@@ -241,5 +249,6 @@
     <xacro:wheel lr_prefix="${lr_prefix}" fr_prefix="${fr_prefix}"
                  lr_reflect="${lr_reflect}" tire_width="${tire_width}"
-                 wheel_mass="${wheel_mass}"/>
+                 wheel_mass="${wheel_mass}"
+                 axle_eff_limit="${axle_eff_limit}"/>
   </xacro:macro>
   <!-- base_link must have geometry so that its axes can be displayed in
@@ -285,5 +294,5 @@
     <material>Gazebo/Grey</material>
     <mu1>0.3</mu1>
-    <mu2>0.3</mu2>
+    <mu2>0.4</mu2>
   </gazebo>
   <joint name="base_link_to_chasis" type="fixed">
@@ -381,17 +390,21 @@
                      lr_reflect="1" fr_reflect="1"
                      tire_width="${front_tire_width}"
-                     wheel_mass="${front_wheel_mass}"/>
+                     wheel_mass="${front_wheel_mass}"
+                     axle_eff_limit="${front_axle_eff_limit}"/>
   <xacro:front_wheel lr_prefix="right" fr_prefix="front"
                      lr_reflect="-1" fr_reflect="1"
                      tire_width="${front_tire_width}"
-                     wheel_mass="${front_wheel_mass}"/>
+                     wheel_mass="${front_wheel_mass}"
+                     axle_eff_limit="${front_axle_eff_limit}"/>
   <xacro:rear_wheel lr_prefix="left" fr_prefix="rear"
                     lr_reflect="1" fr_reflect="-1"
                     tire_width="${rear_tire_width}"
-                    wheel_mass="${rear_wheel_mass}"/>
+                    wheel_mass="${rear_wheel_mass}"
+                    axle_eff_limit="${rear_axle_eff_limit}"/>
   <xacro:rear_wheel lr_prefix="right" fr_prefix="rear"
                     lr_reflect="-1" fr_reflect="-1"
                     tire_width="${rear_tire_width}"
-                    wheel_mass="${rear_wheel_mass}"/>
+                    wheel_mass="${rear_wheel_mass}"
+                    axle_eff_limit="${rear_axle_eff_limit}"/>
   <gazebo>
     <plugin name="gazebo_ros_control" filename="libgazebo_ros_control.so"/>
